Commit message: update

File: orne_description/urdf/alpha/orne_alpha.urdf.xacro (robot description, xacro)
@@ -80,5 +80,5 @@
   <!-- Setting for levelly fixed 2D URG -->
   <xacro:sensor_hokuyo name="hokuyo" parent="base_link" size="0.05 0.05 0.05">
-      <origin xyz="0.212 0 0.375" rpy="0 0 0"/>
+      <origin xyz="0.212 0 0.40" rpy="0 0 0"/>
   </xacro:sensor_hokuyo>
   <!-- <link name="visual_left_wheel">
